Commit message: replace parameter

File: my_robo_description/my_robo.urdf (robot description, URDF)
Before this commit: robot my_robo, 6 links, 5 joints
Links:
- link base_link: geometry collision box size=${link_width} ${link_depth} ${link_height}; visual box size=${link_width} ${link_depth} ${link_height}
- link left_wheel_link: geometry collision cylinder length=${wheel_length} radius=${wheel_radius}; visual cylinder length=${wheel_length} radius=${wheel_radius}
- link right_wheel_link: geometry collision cylinder length=${wheel_length} radius=${wheel_radius}; visual cylinder length=${wheel_length} radius=${wheel_radius}

Commit message: inertia

File: my_robo_description/my_robo.urdf (robot description, URDF)
Before this commit: robot my_robo, 6 links, 5 joints
Links:
- link base_link: mass 0.500 -> ${base_mass}; geometry collision box size=${base_width} ${base_depth} ${base_height}; visual box size=${base_width} ${base_depth} ${base_height}
- link left_wheel_link: mass 0.500 -> ${wheel_mass}
- link right_wheel_link: mass 0.500 -> ${wheel_mass}

Commit message: fix urdf

File: my_robo_description/my_robo.urdf (robot description, URDF)
Before this commit: robot my_robo, 6 links, 5 joints
Links:
- link base_link: geometry collision box size=${bw} ${bd} ${bh}; visual box size=${bw} ${bd} ${bh}
- link caster_link: mass 0.500 -> ${caster_mass}; geometry collision sphere radius=${cr}; visual sphere radius=${cr}
- link left_wheel_link: geometry collision cylinder length=${wl} radius=${wr}; visual cylinder length=${wl} radius=${wr}
- link right_wheel_link: geometry collision cylinder length=${wl} radius=${wr}; visual cylinder length=${wl} radius=${wr}
Joints:
- joint base_link_joint: origin xyz=0 0 0.100 -> xyz=0 0 0
- joint caster_joint: origin xyz=0.150 0 -0.650 -> xyz=${cx} ${cy} ${-cz}
- joint left_wheel_joint: origin xyz=-0.100 0.230 -0.57 rpy=-1.5707 0 0 -> xyz=${-wx} ${wy} ${-wz} rpy=-1.5707 0 0
- joint right_wheel_joint: origin xyz=-0.100 -0.230 -0.57 rpy=1.5707 0 0 -> xyz=${-wx} ${-wy} ${-wz} rpy=1.5707 0 0

Commit message: ロボットのパラメータを変更した

File: my_robo_description/my_robo.urdf (robot description, URDF)
Before this commit: robot my_robo, 6 links, 5 joints
Links:
- added link head_link, mass ${head_mass}; collision box size=${hw} ${hd} ${hh}; visual box size=${hw} ${hd} ${hh}
- added link neck_link, mass ${neck_mass}; collision box size=${nw} ${nd} ${nh}; visual box size=${nw} ${nd} ${nh}
Joints:
- added joint head_joint: type revolute, parent neck_link, child head_link, origin xyz=${hx} ${hy} ${hz} rpy=0 0 0, axis 0 1 0, limit lower=${-M_PI/180.0*30.0} upper=${M_PI/180.0*30.0} effort=0.5293 velocity=6.159937255
- added joint neck_joint: type fixed, parent base_link, child neck_link, origin xyz=${nx} ${ny} ${nz} rpy=0 0 0, axis 0 1 0
- joint hokuyo_joint: origin xyz=0.2 0 0.07 rpy=0 0 0 -> xyz=${bd/2+0.05} 0 0 rpy=0 0 0

Commit message: より実機に近い形に変更

File: my_robo_description/my_robo.urdf (robot description, URDF)
Before this commit: robot my_robo, 8 links, 7 joints
Links:
- link base_footprint: geometry collision box size=${fw} ${fd} ${fh}; visual box size=${fw} ${fd} ${fh}
Joints:
- joint base_link_joint: origin xyz=0 0 0 -> xyz=${bx} ${by} ${bz}
- joint caster_joint: parent base_link -> base_footprint
- joint hokuyo_joint: origin xyz=${bd/2+0.05} 0 0 rpy=0 0 0 -> xyz=0 0 ${hh/2.0+0.025}  rpy=0 0 0; parent base_link -> head_link

Commit message: 首の横回転ができるように和った

File: my_robo_description/my_robo.urdf (robot description, URDF)
Before this commit: robot my_robo, 8 links, 7 joints
Joints:
- joint neck_joint: axis 0 1 0 -> 0 0 1; limit (none) -> lower=${-M_PI/180.0*30.0} upper=${M_PI/180.0*30.0} effort=0.5293 velocity=6.159937255; type fixed -> revolute

Commit message: 実機の首制御

File: my_robo_description/my_robo.urdf (robot description, URDF)
Before this commit: robot my_robo, 8 links, 7 joints
Joints:
- joint head_joint: limit lower=${-M_PI/180.0*30.0} upper=${M_PI/180.0*30.0} effort=0.5293 velocity=6.159937255 -> lower=${-M_PI/180.0*20.0} upper=${M_PI/180.0*20.0} effort=0.5293 velocity=6.159937255
- joint neck_joint: limit lower=${-M_PI/180.0*30.0} upper=${M_PI/180.0*30.0} effort=0.5293 velocity=6.159937255 -> lower=${-M_PI/180.0*40.0} upper=${M_PI/180.0*40.0} effort=0.5293 velocity=6.159937255

Commit message: RobotHWを一本化

File: my_robo_description/my_robo.urdf (robot description, URDF)
Before this commit: robot my_robo, 8 links, 7 joints
Joints:
- joint hokuyo_joint: origin xyz=0 0 ${hh/2.0+0.025}  rpy=0 0 0 -> xyz=${hd/2.0-0.015} 0 ${hh+0.02}  rpy=0 0 0

Commit message: ロボットの初期位置を設定 シミュレータと実機でnavigationを一発起動できるlaunchファイルを追加

File: my_robo_description/my_robo.urdf (robot description, URDF)
Before this commit: robot my_robo, 8 links, 7 joints
Joints:
- joint head_joint: limit lower=${-M_PI/180.0*20.0} upper=${M_PI/180.0*20.0} effort=100.0 velocity=100.0 -> lower=${-M_PI/180.0*20.0} upper=${M_PI/180.0*20.0} effort=0.5293 velocity=6.159937255; type continuous -> revolute
- joint neck_joint: limit lower=${-M_PI/180.0*40.0} upper=${M_PI/180.0*40.0} effort=100.0 velocity=100.0 -> lower=${-M_PI/180.0*40.0} upper=${M_PI/180.0*40.0} effort=0.5293 velocity=6.159937255; type continuous -> revolute

Commit message: urdfパラメータの調整

File: my_robo_description/my_robo.urdf (robot description, URDF)
Before this commit: robot my_robo, 8 links, 7 joints
Joints:
- joint head_joint: limit lower=${-M_PI/180.0*20.0} upper=${M_PI/180.0*20.0} effort=0.5293 velocity=6.159937255 -> lower=${-M_PI/180.0*20.0} upper=${M_PI/180.0*20.0} effort=100.0 velocity=100.0; type revolute -> continuous
- joint neck_joint: limit lower=${-M_PI/180.0*40.0} upper=${M_PI/180.0*40.0} effort=0.5293 velocity=6.159937255 -> lower=${-M_PI/180.0*40.0} upper=${M_PI/180.0*40.0} effort=100.0 velocity=100.0; type revolute -> continuous

Commit message: パラメタ調整

File: my_robo_description/my_robo.urdf (robot description, URDF)
Before this commit: robot my_robo, 8 links, 7 joints
Links:
- added link foot_link; collision box size=${fw} ${fd} ${fh}; visual box size=${fw} ${fd} ${fh}
- link base_footprint: geometry 
Joints:
- added joint foot_joint: type fixed, parent base_link, child foot_link, origin xyz=${-bx} ${-by} ${-bz}
- joint base_link_joint: origin xyz=${bx} ${by} ${bz} -> xyz=0 0 0
- joint caster_joint: parent base_footprint -> foot_link

Commit message: プログラムOを追加

File: my_robo_description/my_robo.urdf (robot description, URDF)
Before this commit: robot my_robo, 9 links, 8 joints
Links:
- link base_link: geometry collision box size=${bd} ${bw} ${bh}; visual box size=${bd} ${bw} ${bh}
- link foot_link: geometry collision box size=${fd} ${fw} ${fh}; visual box size=${fd} ${fw} ${fh}
- link head_link: geometry collision box size=${hd} ${hw} ${hh}; visual box size=${hd} ${hw} ${hh}
- link neck_link: geometry collision box size=${nd} ${nw} ${nh}; visual box size=${nd} ${nw} ${nh}
Joints:
- joint foot_joint: origin xyz=${-bx} ${-by} ${-bz} -> xyz=${fx} ${fy} ${fz}
- joint left_wheel_joint: origin xyz=${-wx} ${wy} ${-wz} rpy=-1.5707 0 0 -> xyz=${wx} ${-wy} ${-wz} rpy=-1.5707 0 0
- joint right_wheel_joint: origin xyz=${-wx} ${-wy} ${-wz} rpy=1.5707 0 0 -> xyz=${wx} ${wy} ${-wz} rpy=1.5707 0 0

Commit message: tweak parameter

File: my_robo_description/my_robo.urdf (robot description, URDF)
Before this commit: robot my_robo, 9 links, 8 joints
Joints:
- joint left_wheel_joint: origin xyz=${wx} ${-wy} ${-wz} rpy=-1.5707 0 0 -> xyz=${wx} ${wy} ${-wz} rpy=${-M_PI/2} 0 0
- joint right_wheel_joint: origin xyz=${wx} ${wy} ${-wz} rpy=1.5707 0 0 -> xyz=${wx} ${-wy} ${-wz} rpy=${M_PI/2} 0 0

Commit message: urdfパラメータの調整

File: my_robo_description/my_robo.urdf (robot description, URDF)
Before this commit: robot my_robo, 9 links, 8 joints
Joints:
- joint left_wheel_joint: parent base_link -> foot_link
- joint right_wheel_joint: parent base_link -> foot_link

Commit message: inflation_radiusの調整とtail_linkの追加

File: my_robo_description/my_robo.urdf (robot description, URDF)
Before this commit: robot my_robo, 9 links, 8 joints
Links:
- added link tail_link; collision box size=${td} ${tw} ${th}; visual box size=${td} ${tw} ${th}
Joints:
- added joint tail_joint: type fixed, parent foot_link, child tail_link, origin xyz=${tx} ${ty} ${tz}

Commit message: remove namespace "my_robo"

File: my_robo_description/my_robo.urdf (robot description, URDF)
Before this commit: robot my_robo, 10 links, 9 joints
Joints:
- joint base_link_joint: origin xyz=0 0 0 -> xyz=${-fpx} 0 ${-fpz}
- joint left_wheel_joint: origin xyz=${wx} ${wy} ${-wz} rpy=${-M_PI/2} 0 0 -> xyz=${wx} ${wy} ${wz} rpy=${-M_PI/2} 0 0
- joint right_wheel_joint: origin xyz=${wx} ${-wy} ${-wz} rpy=${M_PI/2} 0 0 -> xyz=${wx} ${-wy} ${wz} rpy=${M_PI/2} 0 0

Commit message: パラメータ調整

File: my_robo_description/my_robo.urdf (robot description, URDF)
Before this commit: robot my_robo, 10 links, 9 joints
Joints:
- joint head_joint: origin xyz=${hx} ${hy} ${hz} rpy=0 0 0 -> xyz=${hx} ${hy} ${hz} rpy=0 ${hp} 0
